File: F405_pill_V1.1/F405_pill.kicad_sch (KiCad schematic)
At the start: 50 parts, among them J1 Conn_01x04_Male, J2 Conn_01x04_Male, J4 TYPE-C-31-M-12, U1 STM32F405RGTx, U2 MAX3051EKA+T, U3 LM1117-3.3, U4 STM32F405_pill, U5 HT7550-1, Y1 Crystal_GND24

Commit message: finalizing
Parts:
- C1: LCSC C315248 -> C23733
- C14, C15: LCSC C15195 -> C41851
- C20: LCSC C110055 -> C122257
- C8: LCSC C15195 -> C527024
- D2: LCSC C130723 -> C130719
- D3: LCSC C90692 -> C434445
- J1, J2, U4: now left out of the parts list
- J4: footprint HRO_TYPE-C-31-M-12 -> TYPE-C-31-M-12:HRO_TYPE-C-31-M-12
- R3, R4: LCSC C2960873 -> C60310
- R6: LCSC C2909362 -> C25118
- U5: LCSC (none) -> C16106
Connections:
- net at C14.1, J1.3 (Pin_3), R3.2: now also U2.7 (CANH)
Other:
- note added: "CONFIRM: ridiculously large LDO?"
- note added: "NOTE: Split termination may be unnecessary"
- note removed: "CONFIRM: ridiculously large LDO sized and wired correctly?"
Changed lines of the file:
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@@
     (stroke (width 0) (type default) (color 0 0 0 0))
   )
-  (wire (pts (xy 79.375 164.592) (xy 79.375 162.052))
+  (wire (pts (xy 79.375 162.052) (xy 79.375 164.592))
     (stroke (width 0) (type default) (color 0 0 0 0))
   )
@@
   )
   (wire (pts (xy 26.924 126.873) (xy 36.449 126.873))
+    (stroke (width 0) (type default) (color 0 0 0 0))
+  )
+  (wire (pts (xy 80.645 164.592) (xy 79.375 164.592))
     (stroke (width 0) (type default) (color 0 0 0 0))
   )
@@
     (effects (font (size 2 2)) (justify left bottom))
   )
-  (text "CONFIRM: ridiculously \nlarge LDO sized and\nwired correctly?"
-    (at 124.841 182.88 0)
+  (text "CONFIRM: ridiculously \nlarge LDO?" (at 124.841 182.88 0)
     (effects (font (size 1.27 1.27)) (justify left bottom))
   )
@@
     (effects (font (size 1.27 1.27)) (justify left bottom))
   )
+  (text "NOTE: Split termination may\nbe unnecessary" (at 44.577 187.325 0)
+    (effects (font (size 1.27 1.27)) (justify left bottom))
+  )
   (global_label "DUAL1" (shape input) (at 171.704 49.657 180) (fields_autoplaced)
     (effects (font (size 1.27 1.27)) (justify right))
@@
       (effects (font (size 1.27 1.27)) hide)
     )
-    (property "Datasheet" "https://datasheet.lcsc.com/lcsc/1810191223_Samsung-Electro-Mechanics-CL05B103KB5NNNC_C15195.pdf" (id 3) (at 79.375 179.832 0)
-      (effects (font (size 1.27 1.27)) hide)
-    )
-    (property "LCSC" "C15195" (id 6) (at 79.375 179.832 0)
+    (property "Datasheet" "" (id 3) (at 79.375 179.832 0)
+      (effects (font (size 1.27 1.27)) hide)
+    )
+    (property "LCSC" "C41851" (id 6) (at 79.375 179.832 0)
       (effects (font (size 1.27 1.27)) hide)
     )
@@
   )
   (symbol (lib_id "CCC_ESC_Custom_Symbols:STM32F405_pill") (at 174.244 29.337 0) (unit 1)
-    (in_bom yes) (on_board yes)
+    (in_bom no) (on_board yes)
     (property "Reference" "U4" (id 0) (at 185.928 36.703 0))
     (property "Value" "STM32F405_pill" (id 1) (at 186.69 51.181 90))
@@
       (effects (font (size 1.27 1.27)) hide)
     )
+    (property "LCSC" "C16106" (id 4) (at 136.652 165.862 0)
+      (effects (font (size 1.27 1.27)) hide)
+    )
     (pin "1")
     (pin "2")
@@
   )
   (symbol (lib_id "Connector:Conn_01x04_Male") (at 101.854 132.842 0) (mirror x) (unit 1)
-    (in_bom yes) (on_board yes)
+    (in_bom no) (on_board yes)
     (property "Reference" "J2" (id 0) (at 103.124 123.952 0)
       (effects (font (size 1.27 1.27)) (justify right))
@@
     (property "Reference" "J4" (id 0) (at 172.72 131.699 0))
     (property "Value" "TYPE-C-31-M-12" (id 1) (at 170.18 140.589 0))
-    (property "Footprint" "HRO_TYPE-C-31-M-12" (id 2) (at 172.72 132.969 0)
+    (property "Footprint" "TYPE-C-31-M-12:HRO_TYPE-C-31-M-12" (id 2) (at 172.72 132.969 0)
       (effects (font (size 1.27 1.27)) (justify left bottom) hide)
     )
@@
       (effects (font (size 1.27 1.27)) hide)
     )
-    (property "LCSC" "C315248" (id 6) (at 18.034 130.048 0)
+    (property "LCSC" "C23733" (id 6) (at 18.034 130.048 0)
       (effects (font (size 1.27 1.27)) hide)
     )
@@
       (effects (font (size 1.27 1.27)) hide)
     )
-    (property "LCSC" "C2909362" (id 4) (at 165.989 94.361 0)
+    (property "LCSC" "C25118" (id 4) (at 165.989 94.361 0)
       (effects (font (size 1.27 1.27)) hide)
     )
@@
       (effects (font (size 1.27 1.27)) hide)
     )
-    (property "LCSC" "C2960873" (id 6) (at 69.215 173.482 0)
+    (property "LCSC" "C60310" (id 6) (at 69.215 173.482 0)
       (effects (font (size 1.27 1.27)) hide)
     )
@@
       (effects (font (size 1.27 1.27)) hide)
     )
-    (property "Datasheet" "" (id 3) (at 170.434 98.044 0)
+    (property "Datasheet" "~" (id 3) (at 170.434 98.044 0)
       (effects (font (size 1.27 1.27)) hide)
     )
@@
       (effects (font (size 1.27 1.27)) hide)
     )
-    (property "Datasheet" "https://datasheet.lcsc.com/lcsc/1810191223_Samsung-Electro-Mechanics-CL05B103KB5NNNC_C15195.pdf" (id 3) (at 76.835 165.862 0)
-      (effects (font (size 1.27 1.27)) hide)
-    )
-    (property "LCSC" "C15195" (id 6) (at 76.835 165.862 0)
+    (property "Datasheet" "" (id 3) (at 76.835 165.862 0)
+      (effects (font (size 1.27 1.27)) hide)
+    )
+    (property "LCSC" "C41851" (id 6) (at 76.835 165.862 0)
       (effects (font (size 1.27 1.27)) hide)
     )
@@
       (effects (font (size 1.27 1.27)) hide)
     )
-    (property "LCSC" "C110055" (id 6) (at 225.044 140.97 0)
+    (property "LCSC" "C122257" (id 6) (at 225.044 140.97 0)
       (effects (font (size 1.27 1.27)) hide)
     )
@@
   )
   (symbol (lib_id "Connector:Conn_01x04_Male") (at 48.895 172.212 0) (mirror x) (unit 1)
-    (in_bom yes) (on_board yes) (fields_autoplaced)
+    (in_bom no) (on_board yes) (fields_autoplaced)
     (property "Reference" "J1" (id 0) (at 47.625 170.9419 0)
       (effects (font (size 1.27 1.27)) (justify right))
@@
       (effects (font (size 1.27 1.27)) hide)
     )
-    (property "Datasheet" "https://datasheet.lcsc.com/lcsc/1810191223_Samsung-Electro-Mechanics-CL05B103KB5NNNC_C15195.pdf" (id 3) (at 47.117 144.526 0)
-      (effects (font (size 1.27 1.27)) hide)
-    )
-    (property "LCSC" "C15195" (id 6) (at 47.117 144.526 0)
+    (property "Datasheet" "~" (id 3) (at 47.117 144.526 0)
+      (effects (font (size 1.27 1.27)) hide)
+    )
+    (property "LCSC" "C527024" (id 6) (at 47.117 144.526 0)
       (effects (font (size 1.27 1.27)) hide)
     )
@@
       (effects (font (size 1.27 1.27)) hide)
     )
-    (property "LCSC" "C2960873" (id 6) (at 69.215 165.862 0)
+    (property "LCSC" "C60310" (id 6) (at 69.215 165.862 0)
       (effects (font (size 1.27 1.27)) hide)
     )
@@
       (effects (font (size 1.27 1.27)) hide)
     )
-    (property "LCSC" "C90692" (id 6) (at 35.052 101.346 0)
+    (property "LCSC" "C434445" (id 6) (at 35.052 101.346 0)
       (effects (font (size 1.27 1.27)) hide)
     )
@@
       (effects (font (size 1.27 1.27)) hide)
     )
-    (property "Datasheet" "https://datasheet.lcsc.com/lcsc/2008201033_Foshan-NationStar-Optoelectronics-NCD0402G1_C130723.pdf" (id 3) (at 28.702 101.219 90)
-      (effects (font (size 1.27 1.27)) hide)
-    )
-    (property "LCSC" "C130723" (id 6) (at 28.702 101.219 0)
+    (property "Datasheet" "~" (id 3) (at 28.702 101.219 90)
+      (effects (font (size 1.27 1.27)) hide)
+    )
+    (property "LCSC" "C130719" (id 6) (at 28.702 101.219 0)
       (effects (font (size 1.27 1.27)) hide)
     )
@@
     )
     (path "/1eb2cfb1-654e-4304-9c92-8c390f8b426a"
-      (reference "J4") (unit 1) (value "TYPE-C-31-M-12") (footprint "HRO_TYPE-C-31-M-12")
+      (reference "J4") (unit 1) (value "TYPE-C-31-M-12") (footprint "TYPE-C-31-M-12:HRO_TYPE-C-31-M-12")
     )
     (path "/a745e779-85b1-40b9-bada-1ff2fde4de45"
